File: hardware/ECE 299 Project.kicad_sch (KiCad schematic)
At the start: 1 part

Commit message: test commit
Other:
- added sheet Power (Power.kicad_sch)
Changed lines of the file:
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@@
+		)
+	)
+	(sheet
+		(at 203.2 99.06)
+		(size 69.85 31.75)
+		(exclude_from_sim no)
+		(in_bom yes)
+		(on_board yes)
+		(dnp no)
+		(fields_autoplaced yes)
+		(stroke
+			(width 0.1524)
+			(type solid)
+		)
+		(fill
+			(color 0 0 0 0.0000)
+		)
+		(property "Sheetname" "Power"
+			(at 203.2 98.3484 0)
+			(show_name yes)
+			(effects
+				(font
+					(size 1.27 1.27)
+				)
+				(justify left bottom)
+			)
+		)
+		(property "Sheetfile" "Power.kicad_sch"
+			(at 203.2 131.3946 0)
+			(effects
+				(font
+					(size 1.27 1.27)
+				)
+				(justify left top)
+			)
+		)
+		(instances
+			(project "ECE 299 Project"
+				(path "/adf646d2-aa7c-4345-9423-7107505b3b06"
+					(page "2")
+				)
+			)
 		)
 	)
