File: hardware/Main.kicad_sch (KiCad schematic)
At the start: 16 parts, among them SW1 Bourns PEC11R, SW2 Bourns PEC11R, U3 RPi_Pico_TH

Commit message: Rough Board Layout
Parts:
- C5, C6, C7, C8: value 0.01u -> 0.01uF; footprint (none) -> Capacitor_SMD:C_1812_4532Metric
- DISP1: footprint (none) -> Connector_PinHeader_2.00mm:PinHeader_1x07_P2.00mm_Vertical
- R10, R11, R12, R5, R6, R7, R8, R9: value 10k -> 10kΩ; footprint (none) -> Resistor_SMD:R_1812_4532Metric
Changed lines of the file:
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@@
 			)
 		)
-		(property "Value" "10k"
+		(property "Value" "10kΩ"
 			(at 56.896 53.086 0)
 			(effects
@@
 			)
 		)
-		(property "Footprint" ""
+		(property "Footprint" "Resistor_SMD:R_1812_4532Metric"
 			(at 53.594 51.816 90)
 			(effects
@@
 			)
 		)
-		(property "Footprint" ""
+		(property "Footprint" "Connector_PinHeader_2.00mm:PinHeader_1x07_P2.00mm_Vertical"
 			(at 181.61 43.18 0)
 			(effects
@@
 			)
 		)
-		(property "Value" "10k"
+		(property "Value" "10kΩ"
 			(at 62.992 134.366 90)
 			(effects
@@
 			)
 		)
-		(property "Footprint" ""
+		(property "Footprint" "Resistor_SMD:R_1812_4532Metric"
 			(at 59.944 134.874 90)
 			(effects
@@
 			)
 		)
-		(property "Value" "0.01u"
+		(property "Value" "0.01uF"
 			(at 65.786 40.132 90)
 			(effects
@@
 			)
 		)
-		(property "Footprint" ""
+		(property "Footprint" "Capacitor_SMD:C_1812_4532Metric"
 			(at 60.96 41.91 0)
 			(effects
@@
 			)
 		)
-		(property "Value" "10k"
+		(property "Value" "10kΩ"
 			(at 63.754 150.876 90)
 			(effects
@@
 			)
 		)
-		(property "Footprint" ""
+		(property "Footprint" "Resistor_SMD:R_1812_4532Metric"
 			(at 59.944 146.304 90)
 			(effects
@@
 			)
 		)
-		(property "Value" "10k"
+		(property "Value" "10kΩ"
 			(at 63.246 59.69 90)
 			(effects
@@
 			)
 		)
-		(property "Footprint" ""
+		(property "Footprint" "Resistor_SMD:R_1812_4532Metric"
 			(at 59.944 59.944 90)
 			(effects
@@
 			)
 		)
-		(property "Value" "10k"
+		(property "Value" "10kΩ"
 			(at 56.134 83.82 0)
 			(effects
@@
 			)
 		)
-		(property "Footprint" ""
+		(property "Footprint" "Resistor_SMD:R_1812_4532Metric"
 			(at 53.594 82.296 90)
 			(effects
@@
 			)
 		)
-		(property "Value" "0.01u"
+		(property "Value" "0.01uF"
 			(at 65.786 165.862 90)
 			(effects
@@
 			)
 		)
-		(property "Footprint" ""
+		(property "Footprint" "Capacitor_SMD:C_1812_4532Metric"
 			(at 60.96 167.64 0)
 			(effects
@@
 			)
 		)
-		(property "Value" "0.01u"
+		(property "Value" "0.01uF"
 			(at 66.294 91.948 90)
 			(effects
@@
 			)
 		)
-		(property "Footprint" ""
+		(property "Footprint" "Capacitor_SMD:C_1812_4532Metric"
 			(at 60.96 93.98 0)
 			(effects
@@
 			)
 		)
-		(property "Value" "10k"
+		(property "Value" "10kΩ"
 			(at 64.262 76.962 90)
 			(effects
@@
 			)
 		)
-		(property "Footprint" ""
+		(property "Footprint" "Resistor_SMD:R_1812_4532Metric"
 			(at 59.944 72.644 90)
 			(effects
@@
 			)
 		)
-		(property "Value" "10k"
+		(property "Value" "10kΩ"
 			(at 57.15 126.9999 0)
 			(effects
@@
 			)
 		)
-		(property "Footprint" ""
+		(property "Footprint" "Resistor_SMD:R_1812_4532Metric"
 			(at 53.594 125.476 90)
 			(effects
@@
 			)
 		)
-		(property "Value" "0.01u"
+		(property "Value" "0.01uF"
 			(at 66.04 113.792 90)
 			(effects
@@
 			)
 		)
-		(property "Footprint" ""
+		(property "Footprint" "Capacitor_SMD:C_1812_4532Metric"
 			(at 60.96 115.57 0)
 			(effects
@@
 			)
 		)
-		(property "Value" "10k"
+		(property "Value" "10kΩ"
 			(at 57.15 157.4799 0)
 			(effects
@@
 			)
 		)
-		(property "Footprint" ""
+		(property "Footprint" "Resistor_SMD:R_1812_4532Metric"
 			(at 53.594 155.956 90)
 			(effects

Commit message: Revised PCB Layout
Connections:
- net DISP_CS: now also U3.17 (GP13); no longer U3.7 (GP5)
- net DISP_DC: now also U3.16 (GP12); no longer U3.10 (GP7)
- net DISP_RES: now also U3.15 (GP11); no longer U3.9 (GP6)
- net DISP_SCLK: now also U3.19 (GP14); no longer U3.4 (GP2)
- net DISP_SDA: now also U3.20 (GP15); no longer U3.5 (GP3)
- net ENC1A: now also U3.22 (GP17); no longer U3.19 (GP14)
- net ENC1B: now also U3.24 (GP18); no longer U3.20 (GP15)
- net ENC1_BTN: now also U3.21 (GP16); no longer U3.27 (GP21)
- net ENC2A: now also U3.27 (GP21); no longer U3.1 (GP0)
- net ENC2B: now also U3.29 (GP22); no longer U3.2 (GP1)
- net ENC2_BTN: now also U3.26 (GP20); no longer U3.29 (GP22)
- net Radio-Audio/Radio_SCL: now also U3.31 (GP26/ADC0); no longer U3.22 (GP17)
- net Radio-Audio/Radio_SDA: now also U3.32 (GP27/ADC1); no longer U3.21 (GP16)
- no-connect marks 17 -> 15
Changed lines of the file:
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@@
 	)
 	(no_connect
-		(at 140.97 109.22)
+		(at 105.41 99.06)
 	)
 	(no_connect
-		(at 105.41 111.76)
+		(at 105.41 104.14)
 	)
 	(no_connect
-		(at 105.41 104.14)
+		(at 105.41 86.36)
 	)
 	(no_connect
-		(at 140.97 111.76)
+		(at 105.41 81.28)
 	)
 	(no_connect
-		(at 140.97 93.98)
+		(at 105.41 93.98)
 	)
 	(no_connect
-		(at 105.41 99.06)
+		(at 140.97 87.63)
 	)
 	(no_connect
-		(at 140.97 106.68)
+		(at 105.41 91.44)
 	)
 	(no_connect
-		(at 140.97 87.63)
+		(at 105.41 101.6)
 	)
 	(no_connect
@@
 	)
 	(no_connect
-		(at 105.41 109.22)
+		(at 105.41 83.82)
 	)
 	(no_connect
@@
 	)
 	(no_connect
-		(at 140.97 78.74)
-	)
-	(no_connect
-		(at 105.41 101.6)
-	)
-	(no_connect
-		(at 105.41 106.68)
+		(at 105.41 96.52)
 	)
 	(no_connect
-		(at 140.97 96.52)
+		(at 140.97 78.74)
 	)
 	(wire
@@
 	(wire
 		(pts
-			(xy 54.61 121.92) (xy 54.61 115.57)
+			(xy 140.97 93.98) (xy 152.4 93.98)
 		)
 		(stroke
@@
 	(wire
 		(pts
-			(xy 101.6 116.84) (xy 105.41 116.84)
+			(xy 54.61 121.92) (xy 54.61 115.57)
 		)
 		(stroke
@@
 	(wire
 		(pts
-			(xy 140.97 104.14) (xy 144.78 104.14)
+			(xy 144.78 111.76) (xy 140.97 111.76)
 		)
 		(stroke
@@
 	(wire
 		(pts
-			(xy 54.61 93.98) (xy 57.15 93.98)
+			(xy 140.97 116.84) (xy 144.78 116.84)
 		)
 		(stroke
@@
 	(wire
 		(pts
-			(xy 64.77 135.89) (xy 64.77 147.32)
+			(xy 54.61 93.98) (xy 57.15 93.98)
 		)
 		(stroke
@@
 	(wire
 		(pts
-			(xy 165.1 40.64) (xy 170.18 40.64)
+			(xy 64.77 135.89) (xy 64.77 147.32)
 		)
 		(stroke
@@
 	(wire
 		(pts
-			(xy 165.1 38.1) (xy 170.18 38.1)
+			(xy 165.1 40.64) (xy 170.18 40.64)
 		)
 		(stroke
@@
 	(wire
 		(pts
-			(xy 123.19 53.34) (xy 128.27 53.34)
+			(xy 165.1 38.1) (xy 170.18 38.1)
 		)
 		(stroke
@@
 	(wire
 		(pts
-			(xy 140.97 116.84) (xy 149.86 116.84)
+			(xy 123.19 53.34) (xy 128.27 53.34)
 		)
 		(stroke
@@
 	(wire
 		(pts
-			(xy 101.6 78.74) (xy 105.41 78.74)
+			(xy 144.78 104.14) (xy 140.97 104.14)
 		)
 		(stroke
@@
 	(wire
 		(pts
-			(xy 101.6 86.36) (xy 105.41 86.36)
+			(xy 101.6 116.84) (xy 105.41 116.84)
 		)
 		(stroke
@@
 	(wire
 		(pts
-			(xy 101.6 91.44) (xy 105.41 91.44)
+			(xy 101.6 111.76) (xy 105.41 111.76)
 		)
 		(stroke
@@
 	(wire
 		(pts
-			(xy 101.6 81.28) (xy 105.41 81.28)
+			(xy 144.78 101.6) (xy 140.97 101.6)
 		)
 		(stroke
@@
 	(wire
 		(pts
-			(xy 101.6 114.3) (xy 105.41 114.3)
+			(xy 144.78 114.3) (xy 140.97 114.3)
 		)
 		(stroke
@@
 	(wire
 		(pts
-			(xy 101.6 96.52) (xy 105.41 96.52)
+			(xy 101.6 109.22) (xy 105.41 109.22)
 		)
 		(stroke
@@
 	(wire
 		(pts
-			(xy 140.97 114.3) (xy 149.86 114.3)
-		)
-		(stroke
-			(width 0)
-			(type default)
-		)
-	)
-	(wire
-		(pts
 			(xy 45.72 149.86) (xy 45.72 151.13)
 		)
@@
 	(wire
 		(pts
-			(xy 101.6 93.98) (xy 105.41 93.98)
+			(xy 101.6 106.68) (xy 105.41 106.68)
 		)
 		(stroke
@@
 	(wire
 		(pts
-			(xy 101.6 83.82) (xy 105.41 83.82)
+			(xy 101.6 114.3) (xy 105.41 114.3)
 		)
 		(stroke
@@
 	(wire
 		(pts
+			(xy 140.97 96.52) (xy 152.4 96.52)
+		)
+		(stroke
+			(width 0)
+			(type default)
+		)
+	)
+	(wire
+		(pts
 			(xy 49.53 50.8) (xy 45.72 50.8)
 		)
@@
 	(wire
 		(pts
-			(xy 140.97 101.6) (xy 144.78 101.6)
+			(xy 140.97 106.68) (xy 144.78 106.68)
 		)
 		(stroke
@@
 	)
 	(label "ENC1B"
-		(at 101.6 116.84 180)
+		(at 144.78 111.76 0)
 		(effects
 			(font
 				(size 1.27 1.27)
 			)
-			(justify right bottom)
+			(justify left bottom)
 		)
 	)
@@
 	)
 	(label "DISP_SDA"
-		(at 101.6 86.36 180)
+		(at 101.6 116.84 180)
 		(effects
 			(font
@@
 	)
 	(label "ENC1_BTN"
-		(at 144.78 104.14 0)
+		(at 144.78 116.84 0)
 		(effects
 			(font
@@
 	)
 	(label "ENC2_BTN"
-		(at 144.78 101.6 0)
+		(at 144.78 106.68 0)
 		(effects
 			(font
@@
 	)
 	(label "ENC2A"
-		(at 101.6 78.74 180)
+		(at 144.78 104.14 0)
 		(effects
 			(font
 				(size 1.27 1.27)
 			)
-			(justify right bottom)
+			(justify left bottom)
 		)
 	)
@@
 	)
 	(label "ENC1A"
-		(at 101.6 114.3 180)
+		(at 144.78 114.3 0)
 		(effects
 			(font
 				(size 1.27 1.27)
 			)
-			(justify right bottom)
+			(justify left bottom)
 		)
 	)
@@
 	)
 	(label "ENC2B"
-		(at 101.6 81.28 180)
+		(at 144.78 101.6 0)
 		(effects
 			(font
 				(size 1.27 1.27)
 			)
-			(justify right bottom)
+			(justify left bottom)
 		)
 	)
 	(label "DISP_RES"
-		(at 101.6 93.98 180)
+		(at 101.6 106.68 180)
 		(effects
 			(font
@@
 	)
 	(label "DISP_DC"
-		(at 101.6 96.52 180)
+		(at 101.6 109.22 180)
 		(effects
 			(font
@@
 	)
 	(label "DISP_SCLK"
-		(at 101.6 83.82 180)
+		(at 101.6 114.3 180)
 		(effects
 			(font
@@
 	)
 	(label "DISP_CS"
-		(at 101.6 91.44 180)
+		(at 101.6 111.76 180)
 		(effects
 			(font
@@
 	)
 	(sheet
-		(at 149.86 111.125)
+		(at 152.4 90.805)
 		(size 14.605 8.89)
 		(exclude_from_sim no)
@@
 		)
 		(property "Sheetname" "Radio-Audio"
-			(at 149.86 110.4134 0)
+			(at 152.4 90.0934 0)
 			(effects
 				(font
@@
 		)
 		(property "Sheetfile" "Radio-Audio.kicad_sch"
-			(at 149.86 120.5996 0)
+			(at 152.4 100.2796 0)
 			(effects
 				(font
@@
 		)
 		(pin "Radio_SDA" input
-			(at 149.86 116.84 180)
+			(at 152.4 93.98 180)
 			(effects
 				(font
@@
 		)
 		(pin "Radio_SCL" input
-			(at 149.86 114.3 180)
+			(at 152.4 96.52 180)
 			(effects
 				(font

Commit message: Reduced Component Sizes + Added Mounting Holes
Parts:
- C5, C6, C7, C8: footprint Capacitor_SMD:C_1812_4532Metric -> Capacitor_SMD:C_1206_3216Metric
- R10, R11, R12, R5, R6, R7, R8, R9: footprint Resistor_SMD:R_1812_4532Metric -> Resistor_SMD:R_1206_3216Metric
Changed lines of the file:
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@@
 			)
 		)
-		(property "Footprint" "Resistor_SMD:R_1812_4532Metric"
+		(property "Footprint" "Resistor_SMD:R_1206_3216Metric"
 			(at 53.594 51.816 90)
 			(effects
@@
 			)
 		)
-		(property "Footprint" "Resistor_SMD:R_1812_4532Metric"
+		(property "Footprint" "Resistor_SMD:R_1206_3216Metric"
 			(at 59.944 134.874 90)
 			(effects
@@
 			)
 		)
-		(property "Footprint" "Capacitor_SMD:C_1812_4532Metric"
+		(property "Footprint" "Capacitor_SMD:C_1206_3216Metric"
 			(at 60.96 41.91 0)
 			(effects
@@
 			)
 		)
-		(property "Footprint" "Resistor_SMD:R_1812_4532Metric"
+		(property "Footprint" "Resistor_SMD:R_1206_3216Metric"
 			(at 59.944 146.304 90)
 			(effects
@@
 			)
 		)
-		(property "Footprint" "Resistor_SMD:R_1812_4532Metric"
+		(property "Footprint" "Resistor_SMD:R_1206_3216Metric"
 			(at 59.944 59.944 90)
 			(effects
@@
 			)
 		)
-		(property "Footprint" "Resistor_SMD:R_1812_4532Metric"
+		(property "Footprint" "Resistor_SMD:R_1206_3216Metric"
 			(at 53.594 82.296 90)
 			(effects
@@
 			)
 		)
-		(property "Footprint" "Capacitor_SMD:C_1812_4532Metric"
+		(property "Footprint" "Capacitor_SMD:C_1206_3216Metric"
 			(at 60.96 167.64 0)
 			(effects
@@
 			)
 		)
-		(property "Footprint" "Capacitor_SMD:C_1812_4532Metric"
+		(property "Footprint" "Capacitor_SMD:C_1206_3216Metric"
 			(at 60.96 93.98 0)
 			(effects
@@
 			)
 		)
-		(property "Footprint" "Resistor_SMD:R_1812_4532Metric"
+		(property "Footprint" "Resistor_SMD:R_1206_3216Metric"
 			(at 59.944 72.644 90)
 			(effects
@@
 			)
 		)
-		(property "Footprint" "Resistor_SMD:R_1812_4532Metric"
+		(property "Footprint" "Resistor_SMD:R_1206_3216Metric"
 			(at 53.594 125.476 90)
 			(effects
@@
 			)
 		)
-		(property "Footprint" "Capacitor_SMD:C_1812_4532Metric"
+		(property "Footprint" "Capacitor_SMD:C_1206_3216Metric"
 			(at 60.96 115.57 0)
 			(effects
@@
 			)
 		)
-		(property "Footprint" "Resistor_SMD:R_1812_4532Metric"
+		(property "Footprint" "Resistor_SMD:R_1206_3216Metric"
 			(at 53.594 155.956 90)
 			(effects
