File: hardware/Radio-Audio.kicad_sch (KiCad schematic)
At the start: 20 parts, among them U1 LM386, U2 RDA5807M_Module

Commit message: Repositioned + Added volume potentiometer to PMW Audio
Parts:
- removed R17: 0 ohm, symbol Device:R_US
- removed U2: RDA5807M_Module, ECE:RDA5807M_Module_SM, symbol ECE:RDA5807M_Module
- added RV2: 10kΩ, Potentiometer_SMD:Potentiometer_Bourns_3314J_Vertical, symbol Device:R_Potentiometer_Trim_US
- added U5: RDA5807M_Module, ECE:RDA5807M_Module_SM, symbol ECE:RDA5807M_Module
- C11, C12: footprint (none) -> Capacitor_SMD:C_1206_3216Metric
- R13, R14, R15, R16: footprint (none) -> Resistor_SMD:R_1206_3216Metric
Connections:
- net +3.3V: now also U5.5 (VDD)
- net GND: now also RV2.3, U5.6 (GND)
- net Radio_SCL: now also U5.2 (SCLK)
- net Radio_SDA: now also U5.1 (SDIO)
- net at RV1.2: now also U5.7 (ROUT)
- net at AE1.1 (A): now also U5.10 (FMIN)
- net at C4.2, R2.1: now also R16.2, U1.3 (+)
- net at C12.1, R15.2: now also RV2.2; no longer R16.1
- new net: R16.1, RV2.1
Other:
- moved on the sheet: C11, C12, R13, R14, R15

Commit message: Did it all lmao (pcb traces ready for full review)
Parts:
- added R17, R18: 0 ohm, Resistor_SMD:R_1206_3216Metric, symbol Device:R_US
- LS1: footprint Connector_PinHeader_2.00mm:PinHeader_1x02_P2.00mm_Vertical -> TerminalBlock:TerminalBlock_MaiXu_MX126-5.0-02P_1x02_P5.00mm
Connections:
- net at AE1.1 (A), U5.10 (FMIN): now also R18.1
- net at C4.2, R2.1: now also R17.1; no longer R16.2, U1.3 (+)
- new net: R16.2, R17.2, U1.3 (+)
- new net Board Antenna: R18.2
Changed lines of the file:
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@@
+	)
+	(junction
+		(at 113.03 80.01)
+		(diameter 0)
+		(color 0 0 0 0)
+	)
+	(junction
+		(at 144.78 93.98)
+		(diameter 0)
+		(color 0 0 0 0)
 	)
 	(junction
@@
 	)
 	(junction
-		(at 144.78 93.98)
-		(diameter 0)
-		(color 0 0 0 0)
-	)
-	(junction
 		(at 66.04 92.71)
 		(diameter 0)
@@
 	(wire
 		(pts
+			(xy 121.92 80.01) (xy 120.65 80.01)
+		)
+		(stroke
+			(width 0)
+			(type default)
+		)
+	)
+	(wire
+		(pts
 			(xy 152.4 80.01) (xy 152.4 93.98)
 		)
@@
 	(wire
 		(pts
-			(xy 144.78 93.98) (xy 152.4 93.98)
-		)
-		(stroke
-			(width 0)
-			(type default)
-		)
-	)
-	(wire
-		(pts
 			(xy 105.41 107.95) (xy 110.49 107.95)
 		)
@@
 	(wire
 		(pts
+			(xy 121.92 81.28) (xy 121.92 80.01)
+		)
+		(stroke
+			(width 0)
+			(type default)
+		)
+	)
+	(wire
+		(pts
 			(xy 121.92 48.26) (xy 125.73 48.26)
 		)
@@
 			(width 0)
 			(type default)
+		)
+	)
+	(label "Board Antenna"
+		(at 121.92 81.28 0)
+		(effects
+			(font
+				(size 1.27 1.27)
+			)
+			(justify left bottom)
 		)
 	)
@@
 	)
 	(symbol
+		(lib_id "Device:R_US")
+		(at 116.84 80.01 90)
+		(unit 1)
+		(exclude_from_sim no)
+		(in_bom yes)
+		(on_board yes)
+		(dnp no)
+		(property "Reference" "R18"
+			(at 118.364 84.582 90)
+			(effects
+				(font
+					(size 1.27 1.27)
+				)
+			)
+		)
+		(property "Value" "0 ohm"
+			(at 118.11 82.55 90)
+			(effects
+				(font
+					(size 1.27 1.27)
+				)
+			)
+		)
+		(property "Footprint" "Resistor_SMD:R_1206_3216Metric"
+			(at 117.094 78.994 90)
+			(effects
+				(font
+					(size 1.27 1.27)
+				)
+				(hide yes)
+			)
+		)
+		(property "Datasheet" "~"
+			(at 116.84 80.01 0)
+			(effects
+				(font
+					(size 1.27 1.27)
+				)
+				(hide yes)
+			)
+		)
+		(property "Description" "Resistor, US symbol"
+			(at 116.84 80.01 0)
+			(effects
+				(font
+					(size 1.27 1.27)
+				)
+				(hide yes)
+			)
+		)
+		(pin "1"
+		)
+		(pin "2"
+		)
+		(instances
+			(project ""
+				(path "/adf646d2-aa7c-4345-9423-7107505b3b06/1b91a94e-3823-4ebf-b09f-64912f681b22"
+					(reference "R18")
+					(unit 1)
+				)
+			)
+		)
+	)
+	(symbol
 		(lib_id "Device:C_US")
 		(at 186.69 107.95 0)
@@
 	)
 	(symbol
+		(lib_id "Device:R_US")
+		(at 148.59 93.98 90)
+		(unit 1)
+		(exclude_from_sim no)
+		(in_bom yes)
+		(on_board yes)
+		(dnp no)
+		(fields_autoplaced yes)
+		(property "Reference" "R17"
+			(at 148.59 87.63 90)
+			(effects
+				(font
+					(size 1.27 1.27)
+				)
+			)
+		)
+		(property "Value" "0 ohm"
+			(at 148.59 90.17 90)
+			(effects
+				(font
+					(size 1.27 1.27)
+				)
+			)
+		)
+		(property "Footprint" "Resistor_SMD:R_1206_3216Metric"
+			(at 148.844 92.964 90)
+			(effects
+				(font
+					(size 1.27 1.27)
+				)
+				(hide yes)
+			)
+		)
+		(property "Datasheet" "~"
+			(at 148.59 93.98 0)
+			(effects
+				(font
+					(size 1.27 1.27)
+				)
+				(hide yes)
+			)
+		)
+		(property "Description" "Resistor, US symbol"
+			(at 148.59 93.98 0)
+			(effects
+				(font
+					(size 1.27 1.27)
+				)
+				(hide yes)
+			)
+		)
+		(pin "1"
+		)
+		(pin "2"
+		)
+		(instances
+			(project ""
+				(path "/adf646d2-aa7c-4345-9423-7107505b3b06/1b91a94e-3823-4ebf-b09f-64912f681b22"
+					(reference "R17")
+					(unit 1)
+				)
+			)
+		)
+	)
+	(symbol
 		(lib_id "Device:C_Polarized_US")
 		(at 204.47 96.52 90)
@@
 			)
 		)
-		(property "Footprint" "Connector_PinHeader_2.00mm:PinHeader_1x02_P2.00mm_Vertical"
+		(property "Footprint" "TerminalBlock:TerminalBlock_MaiXu_MX126-5.0-02P_1x02_P5.00mm"
 			(at 223.52 101.6 0)
 			(effects
